File: board/rocketBoards/mainBoardV1.sch (EAGLE design)
At the start: 47 parts

Commit message: Board layout done with autorouting
Parts:
- removed JP3: M02-JST-2-PTH-NO_SILK, SparkFun-Connectors:M02-JST-2-PTH-NO_SILK
- removed JP4: USB_MICROB_PLUGCONN-11752, SparkFun-Connectors:USB_MICROB_PLUGCONN-11752
- removed S2: DPDT, SparkFun-Electromechanical:SWITCH-DPDTAYZ0202
- added C20, C22, C24, C25, C26: .1uF, ELL-i-Passives:C0402
- added C21: 100uF, ELL-i-Passives:CC1206
- added C27, C28, C29, C30: .01uF, ELL-i-Passives:C0402
- added J1: 47346-0001, ELL-i-Connectors:MICRO-USB
- added JP2: (no value), SparkFun-Connectors:M04JST
- added JP8: M02-JST-2-PTH-NO_SILK, SparkFun-Connectors:M02-JST-2-PTH-NO_SILK
- added R10: (no value), ELL-i-Passives:R0402
- added S4: DPDT, SparkFun-Electromechanical:SWITCH-DPDTAYZ0202
- added U$6: LDK220M33R, Sensors:LDK220M33R
- C10, C14: value 1uF -> 10uF; MPN MC0402X105M6R3CT -> (none); OC_NEWARK 06R4879 -> (none)
- C11, C16: value 0.1uF -> .1uF; OC_NEWARK unknown -> (none)
- C12, C13, C19, C9: value 10uF -> .1uF; OC_NEWARK unknown -> (none)
- C15: value 1uF -> .1uF; MPN MC0402X105M6R3CT -> (none); OC_NEWARK 06R4879 -> (none)
- C17: value 0.1uF -> 1uF; OC_NEWARK unknown -> (none)
- C18: value 10uF -> 1uF; device ELL-i-Passives:CPOL1206 -> ELL-i-Passives:C0402; MPN 293D106X06R3B2TE3 -> (none); OC_NEWARK 99M0346 -> (none)
- C8: device ELL-i-Passives:CPOL1206 -> ELL-i-Passives:C0402; MPN 293D106X06R3B2TE3 -> (none); OC_NEWARK 99M0346 -> (none)
- R1, R4: device ELL-i-Passives:R0402 -> ELL-i-Passives:R0805
- R6: value 33 -> 0; OC_NEWARK unknown -> (none)
- R7: value 33 -> (none); OC_NEWARK unknown -> (none)
Connections:
- removed net USB_FTOGGLE: S2.5, U1.PIO0_1/CLKOUT/CT32B0_MAT2/USB_FTOGGLE
- new net DRDY_M: 9-AXIS.DRDY_M, U1.PIO0_19/U0_TXD/CT32B0_MAT1
- new net LED_PIN2: LED1.A, U1.PIO0_18/U0_RXD/CT32B0_MAT0
- new net N$20: JP8.1, S4.1
- new net N$21: R10.2, U$3.DAT1
- new net PIO0_1: S4.5, U1.PIO0_1/CLKOUT/CT32B0_MAT2/USB_FTOGGLE
- new net SD_CD: U$3.CD, U1.PIO1_21/U0_DCDN/SSP1_MISO/CT16B0_CAP1
- net 3.3V: now also C19.1, C21.1, C22.1, C24.1, C25.1, C26.1, C27.1, C28.1, C29.1, C30.1, C8.1, JP2.1, R10.1, R6.2, R7.2, S4.6, U$6.OUT; no longer 9-AXIS.DEN_A/G, C17.1, C8.+, LED1.A, S2.6
- net GND: now also C18.2, C20.2, C21.2, C22.2, C24.2, C25.2, C26.2, C27.2, C28.2, C29.2, C30.2, C8.2, J1.GND, J1.P1, J1.P2, J1.P3, J1.P4, J1.P5, J1.P6, JP2.3, JP8.2, S4.4, U$6.GND; no longer C18.-, C8.-, JP3.2, JP4.GND, JP4.SHIELD, S2.4
- net N$1: now also 9-AXIS.DEN_A/G, R6.1; no longer JP3.1, S2.1
- net N$14: now also 9-AXIS.C1, C20.1; no longer R6.2, U1.USB_DP
- net N$15: now also J1.D+, U1.USB_DP; no longer JP4.D+, R6.1
- net N$16: now also U$3.DAT2; no longer JP4.D-
- net N$17: now also J1.D-; no longer R7.2
- net SSP1_SSEL: now also U1.PIO1_13/U1_CTSN/SCT0_OUT3/R_22; no longer U1.PIO0_23/ADC_1/R_9/U0_NRI/SSP1_SSEL
- net USB_VBUS: now also J1.VBUS, S4.3; no longer JP4.VCC, S2.3
- net VBUS: now also C17.1, C18.1, JP2.4, S4.2, U$6.EN, U$6.IN; no longer C18.+, C19.1, S2.2
